Commit message: fix

File: module06/ex03/ubot/ubot_description/urdf/robot.urdf.xacro (robot description, xacro)
@@ -215,4 +215,7 @@
                     name="gz::sim::systems::Sensors">
                 <render_engine>ogre2</render_engine>
+        </plugin>
+        <plugin filename="gz-sim-imu-system"
+            name="gz::sim::systems::Imu">
         </plugin>
     </gazebo>
@@ -401,5 +404,5 @@
         <origin xyz="0 0 0"/>
         <geometry>
-            <box size="0.02 0.05 0.05"/>
+            <box size="0.02 1.05 0.05"/>
         </geometry>
     </collision>
@@ -417,3 +420,4 @@
 <!-- ====================== -->
     <!-- END IMU SENSOR -->
+ячё
 </robot>
